File: echo-esphome.kicad_pcb (KiCad board)
At the start: 2 copper layers, 70 x 55.6 mm, 3 parts, among them J1 Conn_01x27_Pin, U1 MAX98357A, U2 M5STAMP-PICO

Commit message: Add measurements
Other:
- board size 70 x 55.6 mm -> 70 x 52.6 mm
Changed lines of the file:
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@@
 	)
 	(gr_circle
-		(center 122.5 120.5)
-		(end 122.5 123.5)
+		(center 125.06 115.5)
+		(end 128.06 115.5)
 		(stroke
 			(width 0.15)
@@
 	)
 	(gr_circle
-		(center 100 99.9)
-		(end 138 99.9)
+		(center 100 100)
+		(end 138 100)
 		(stroke
 			(width 0.1)
@@
 	)
 	(dimension
+		(type radial)
+		(layer "User.2")
+		(pts
+			(xy 100 100) (xy 138 100)
+		)
+		(leader_length 3.81)
+		(gr_text "R 38.0000 mm"
+			(at 154.51 100 0)
+			(layer "User.2")
+			(effects
+				(font
+					(size 1 1)
+					(thickness 0.15)
+				)
+			)
+		)
+		(format
+			(prefix "R ")
+			(suffix "")
+			(units 3)
+			(units_format 1)
+			(precision 4)
+		)
+		(style
+			(thickness 0.1)
+			(arrow_length 1.27)
+			(text_position_mode 0)
+			(extension_offset 0.5) keep_text_aligned)
+	)
+	(dimension
+		(type radial)
+		(layer "User.3")
+		(pts
+			(xy 100 100) (xy 65 100)
+		)
+		(leader_length 3.81)
+		(gr_text "R 35.0000 mm"
+			(at 48.49 100 0)
+			(layer "User.3")
+			(effects
+				(font
+					(size 1 1)
+					(thickness 0.15)
+				)
+			)
+		)
+		(format
+			(prefix "R ")
+			(suffix "")
+			(units 3)
+			(units_format 1)
+			(precision 4)
+		)
+		(style
+			(thickness 0.1)
+			(arrow_length 1.27)
+			(text_position_mode 0)
+			(extension_offset 0.5) keep_text_aligned)
+	)
+	(dimension
+		(type orthogonal)
+		(layer "Edge.Cuts")
+		(pts
+			(xy 125.06 115.5) (xy 125.06 118.5)
+		)
+		(height 16.69)
+		(orientation 1)
+		(gr_text "3.0000 mm"
+			(at 140.6 117 90)
+			(layer "Edge.Cuts")
+			(effects
+				(font
+					(size 1 1)
+					(thickness 0.15)
+				)
+			)
+		)
+		(format
+			(prefix "")
+			(suffix "")
+			(units 3)
+			(units_format 1)
+			(precision 4)
+		)
+		(style
+			(thickness 0.15)
+			(arrow_length 1.27)
+			(text_position_mode 0)
+			(extension_height 0.58642)
+			(extension_offset 0.5) keep_text_aligned)
+	)
+	(dimension
+		(type orthogonal)
+		(layer "User.1")
+		(pts
+			(xy 125.06 115.5) (xy 125 120.5)
+		)
+		(height -5.06)
+		(orientation 1)
+		(gr_text "5.0000 mm"
+			(at 118.85 118 90)
+			(layer "User.1")
+			(effects
+				(font
+					(size 1 1)
+					(thickness 0.15)
+				)
+			)
+		)
+		(format
+			(prefix "")
+			(suffix "")
+			(units 3)
+			(units_format 1)
+			(precision 4)
+		)
+		(style
+			(thickness 0.1)
+			(arrow_length 1.27)
+			(text_position_mode 0)
+			(extension_height 0.58642)
+			(extension_offset 0.5) keep_text_aligned)
+	)
+	(dimension
 		(type orthogonal)
 		(layer "User.4")
@@
 			(effects
 				(font
+					(size 1 1)
+					(thickness 0.15)
+				)
+			)
+		)
+		(format
+			(prefix "")
+			(suffix "")
+			(units 3)
+			(units_format 1)
+			(precision 4)
+		)
+		(style
+			(thickness 0.1)
+			(arrow_length 1.27)
+			(text_position_mode 0)
+			(extension_height 0.58642)
+			(extension_offset 0.5) keep_text_aligned)
+	)
+	(dimension
+		(type orthogonal)
+		(layer "User.9")
+		(pts
+			(xy 84 61.9) (xy 84 67.9)
+		)
+		(height -6.5)
+		(orientation 1)
+		(gr_text "6.0000 mm"
+			(at 76.35 64.9 90)
+			(layer "User.9")
+			(effects
+				(font
